File: KiCad/FA-ADC.kicad_pcb (KiCad board)
At the start: 2 copper layers, 80 x 43 mm, 124 parts, among them J100 Conn_02x10_Odd_Even, J101 Conn_01x03_Male, J102 Conn_01x02_Male, J103 Conn_01x02_Male, J104 Conn_01x02_Male, J105 Conn_01x02_Male, U200 AD1974, U300 AD797, U301 AD797, U400 AD797, U401 AD797, U500 AD797, U501 AD797, U600 AD797, U601 AD797, Y200 12.288MHz

Commit message: Update for release
Parts:
- removed C211, C212: 22p, Capacitor_SMD:C_0402_1005Metric
- removed J104, J105: Conn_01x02_Male, Connector_JST:JST_PH_B2B-PH-SM4-TB_1x02-1MP_P2.00mm_Vertical
- removed NT1: Net-Tie_2, NetTie:NetTie-2_SMD_Pad0.5mm
- removed R201: 0R, Resistor_SMD:R_0402_1005Metric
- removed R202: 49.9R, Resistor_SMD:R_0402_1005Metric
- removed Y200: 12.288MHz, Crystal:Crystal_SMD_5032-4Pin_5.0x3.2mm
- added C1: 4.7u, Capacitor_SMD:C_0402_1005Metric, F.Cu at (-29.8, 15.2)
- added C2: 100n, Capacitor_SMD:C_0402_1005Metric, F.Cu at (-29.8, 14.2)
- added C3: 10n, Capacitor_SMD:C_0402_1005Metric, F.Cu at (-29.8, 7.25)
- added C4: 1u, Capacitor_SMD:C_0402_1005Metric, F.Cu at (-29.8, 6.25)
- added D300: TBD, Diode_SMD:D_0402_1005Metric, F.Cu at (27.0, 15.8)
- added D400: TBD, Diode_SMD:D_0402_1005Metric, F.Cu at (27.0, 5.00)
- added D500: TBD, Diode_SMD:D_0402_1005Metric, F.Cu at (27.0, -4.75)
- added D600: TBD, Diode_SMD:D_0402_1005Metric, F.Cu at (27.0, -15.5)
- added FB300: 600R, Inductor_SMD:L_0402_1005Metric, F.Cu at (27.0, 16.8)
- added FB400: 600R, Inductor_SMD:L_0402_1005Metric, F.Cu at (27.0, 6.00)
- added FB500: 600R, Inductor_SMD:L_0402_1005Metric, F.Cu at (27.0, -5.75)
- added FB600: 600R, Inductor_SMD:L_0402_1005Metric, F.Cu at (27.0, -16.5)
- added J1: TC2030, Connector:Tag-Connect_TC2030-IDC-NL_2x03_P1.27mm_Vertical, B.Cu at (-20.5, 18.0)
- added R1: 2.2k, Resistor_SMD:R_0402_1005Metric, F.Cu at (-28.8, 3.25)
- added R10: 0R, Resistor_SMD:R_0402_1005Metric, F.Cu at (-24.8, 8.50)
- added R11: 100R, Resistor_SMD:R_0402_1005Metric, F.Cu at (-24.7, 15.6)
- added R12: 0R, Resistor_SMD:R_0402_1005Metric, F.Cu at (-28.2, 14.8)
- added R13: 0R, Resistor_SMD:R_0402_1005Metric, F.Cu at (-27.2, 14.8)
- added R14: 100R, Resistor_SMD:R_0402_1005Metric, F.Cu at (-24.7, 14.6)
- added R15: 100R, Resistor_SMD:R_0402_1005Metric, F.Cu at (-24.7, 13.6)
- added R16: 0R, Resistor_SMD:R_0402_1005Metric, F.Cu at (-24.8, 7.50)
- added R2: 2.2k, Resistor_SMD:R_0402_1005Metric, F.Cu at (-28.8, 5.25)
- added R3: 100R, Resistor_SMD:R_0402_1005Metric, F.Cu at (-27.2, 6.75)
- added R4: 100R, Resistor_SMD:R_0402_1005Metric, F.Cu at (-28.2, 6.75)
- added R5: 100R, Resistor_SMD:R_0402_1005Metric, F.Cu at (-24.8, 11.5)
- added R6: 100R, Resistor_SMD:R_0402_1005Metric, F.Cu at (-24.8, 10.5)
- added R7: 100R, Resistor_SMD:R_0402_1005Metric, F.Cu at (-24.8, 9.50)
- added R8: 10k, Resistor_SMD:R_0402_1005Metric, F.Cu at (-26.2, 6.75)
- added R9: 100R, Resistor_SMD:R_0402_1005Metric, F.Cu at (-24.8, 12.5)
- added U100: STM32F042G4Ux, Package_DFN_QFN:QFN-28_4x4mm_P0.5mm, F.Cu at (-28.8, 10.8)
- C205: value 2.2n -> 390p
- C206: value 39n -> 5.6n
- J101: value Conn_01x03_Male -> JST_XH_S3B; footprint Connector_JST:JST_PH_B3B-PH-SM4-TB_1x03-1MP_P2.00mm_Vertical -> Connector_JST:JST_XH_S3B-XH-A_1x03_P2.50mm_Horizontal
- J102: value Conn_01x02_Male -> JST_XH_S8B; footprint Connector_JST:JST_PH_B2B-PH-SM4-TB_1x02-1MP_P2.00mm_Vertical -> Connector_JST:JST_XH_S8B-XH-A_1x08_P2.50mm_Horizontal
- J103: value Conn_01x02_Male -> USB_OTG; footprint Connector_JST:JST_PH_B2B-PH-SM4-TB_1x02-1MP_P2.00mm_Vertical -> Connector_USB:USB_Micro-B_Molex-105017-0001
- PCB100: value Board_Module -> 70x43
- R200: value 3.32k -> 562R
- moved J101 218.9 mm to (-20.0, 12.2), turned to 0 degrees
- moved J103 217.8 mm to (-28.0, 18.8), turned to 0 degrees
- moved J100 174.4 mm to (-33.2, 11.4)
- moved PCB100 174.4 mm to (0.00, 0.00)
- moved J102 174.0 mm to (30.6, 8.75), turned to 90 degrees
- moved FB201 171.0 mm to (-26.2, -6.50), turned to 270 degrees
- moved C205 170.2 mm to (-15.0, -3.25)
- moved C206 170.2 mm to (-14.0, -3.25)
- moved R200 170.2 mm to (-14.5, -4.75)
- moved C305 170.2 mm to (-10.0, 14.0)
- moved C405 170.2 mm to (-10.0, 3.25)
- moved C505 170.2 mm to (-10.0, -7.25)
- moved C605 170.2 mm to (-10.0, -18.0)
- moved C209 170.2 mm to (-17.8, 7.75)
- moved C200 170.1 mm to (-16.5, -4.50)
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Connections:
- net /ADC/I2S_SDIN2 renamed /I2S_SD1
- C200 pad 2: GNDA -> GND
- C201 pad 2: GNDA -> GND
- C202 pad 2: GNDA -> GND
- C203 pad 2: GNDA -> GND
- C207 pad 2: GNDA -> GND
- C208 pad 2: GNDA -> GND
- C209 pad 2: GNDA -> GND
- C210 pad 2: GNDA -> GND
- C300 pad 1: GNDA -> GND
- C300 pad 2: /Left Buffer 1/In -> Net-(C300-Pad2)
- C305 pad 1: GNDA -> GND
- C306 pad 2: GNDA -> GND
- C308 pad 1: GNDA -> GND
- C309 pad 1: GNDA -> GND
- C310 pad 2: GNDA -> GND
- C311 pad 2: GNDA -> GND
- C312 pad 1: GNDA -> GND
- C313 pad 1: GNDA -> GND
- C314 pad 2: GNDA -> GND
- C315 pad 2: GNDA -> GND
- C400 pad 1: GNDA -> GND
- C400 pad 2: /Right Buffer 1/In -> Net-(C400-Pad2)
- C405 pad 1: GNDA -> GND
- C406 pad 2: GNDA -> GND
- C408 pad 1: GNDA -> GND
- C409 pad 1: GNDA -> GND
- C410 pad 2: GNDA -> GND
- C411 pad 2: GNDA -> GND
- C412 pad 1: GNDA -> GND
- C413 pad 1: GNDA -> GND
- C414 pad 2: GNDA -> GND
- C415 pad 2: GNDA -> GND
- C500 pad 1: GNDA -> GND
- C500 pad 2: /Left Buffer 2/In -> Net-(C500-Pad2)
- C505 pad 1: GNDA -> GND
- C506 pad 2: GNDA -> GND
- C508 pad 1: GNDA -> GND
- C509 pad 1: GNDA -> GND
- C510 pad 2: GNDA -> GND
- C511 pad 2: GNDA -> GND
- C512 pad 1: GNDA -> GND
- C513 pad 1: GNDA -> GND
- C514 pad 2: GNDA -> GND
- C515 pad 2: GNDA -> GND
- C600 pad 1: GNDA -> GND
- C600 pad 2: /Right Buffer 2/In -> Net-(C600-Pad2)
- C605 pad 1: GNDA -> GND
- C606 pad 2: GNDA -> GND
- C608 pad 1: GNDA -> GND
- C609 pad 1: GNDA -> GND
- C610 pad 2: GNDA -> GND
- C611 pad 2: GNDA -> GND
- C612 pad 1: GNDA -> GND
- C613 pad 1: GNDA -> GND
- C614 pad 2: GNDA -> GND
- C615 pad 2: GNDA -> GND
- J100 pad 1: /I2S_MCLK -> +3V3
- J100 pad 10: Net-(J100-Pad10) -> GND
- J100 pad 11: /SPI_MISO -> /RESERVED
- J100 pad 12: /SPI_CS -> GND
- J100 pad 13: /SPI_SCK -> /I2S_SD0
- J100 pad 14: /SPI_MOSI -> GND
- J100 pad 15: /SHDN -> /I2S_LRCLK
- J100 pad 16: /MUTE -> GND
- J100 pad 17: GND -> /I2S_BCLK
- J100 pad 19: +3V3 -> /I2S_MCLK
- J100 pad 2: GND -> +5V
- J100 pad 20: +5V -> GND
- J100 pad 3: /I2S_LRCLK -> /nMUTE
- J100 pad 5: /I2S_BCLK -> /ENABLE
- J100 pad 7: /I2S_SDI -> /I2C_SDA
- J100 pad 9: Net-(J100-Pad9) -> /I2C_SCL
- J101 pad 2: GNDA -> GND
- J102 pad 2: GNDA -> GND
- J103 pad 1: /Right Buffer 1/In -> VBUS
- J103 pad 2: GNDA -> /USB_DM
- PCB100 pad 3: GNDA -> GND
- PCB100 pad 4: GNDA -> GND
- R300 pad 2: /Left Buffer 1/In -> Net-(C300-Pad2)
- R400 pad 2: /Right Buffer 1/In -> Net-(C400-Pad2)
- R500 pad 2: /Left Buffer 2/In -> Net-(C500-Pad2)
- R600 pad 2: /Right Buffer 2/In -> Net-(C600-Pad2)
- U200 pad 1: GNDA -> GND
- U200 pad 10: /SHDN -> /ENABLE
- U200 pad 2: Net-(C212-Pad1) -> /I2S_MCLK
- U200 pad 20: /I2S_SDI -> /I2S_SD0
- U200 pad 32: GNDA -> GND
- U200 pad 34: GNDA -> GND
- U200 pad 36: GNDA -> GND
- U200 pad 4: GNDA -> GND
- U300 pad 3: GNDA -> GND
- U301 pad 3: GNDA -> GND
- U400 pad 3: GNDA -> GND
- U401 pad 3: GNDA -> GND
- U500 pad 3: GNDA -> GND
- U501 pad 3: GNDA -> GND
- U600 pad 3: GNDA -> GND
- U601 pad 3: GNDA -> GND
Routing:
- net +15V: track 0.00 -> 187.7 mm, vias 0 -> 1
- net -15V: track 0.00 -> 153.8 mm, vias 0 -> 7
- net +3V3: track 0.00 -> 79.7 mm, vias 0 -> 3
- net /ENABLE: track 0.00 -> 36.7 mm, vias 0 -> 1
- net GND: track 0.00 -> 35.0 mm, vias 0 -> 595
- net Net-(C501-Pad1): track 0.00 -> 29.6 mm, vias 0 -> 2
- net Net-(C601-Pad1): track 0.00 -> 28.8 mm, vias 0 -> 2
- net Net-(C301-Pad1): track 0.00 -> 28.1 mm, vias 0 -> 2
- net Net-(C401-Pad1): track 0.00 -> 28.0 mm, vias 0 -> 2
- net Net-(C200-Pad1): track 0.00 -> 25.8 mm
- net /ADC/In_L0N: track 0.00 -> 22.3 mm
- net /ADC/In_R1N: track 0.00 -> 22.2 mm
- net /ADC/In_L0P: track 0.00 -> 22.2 mm
- net /ADC/In_R1P: track 0.00 -> 21.8 mm
- net /I2S_LRCLK: track 0.00 -> 20.2 mm
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- added copper zone on B.Cu, net GND
- added copper zone on F.Cu, net GND
Other:
- board text added: "Farving Acoustics FA-ADC 1000003-2.0.0"
